File: hardware/charge-hf.kicad_pcb (KiCad board)
At the start: 4 copper layers, 100 x 32 mm, 98 parts, among them J1 USB_C_Receptacle_USB2.0, J10 DEBUG, J11 OLED, J2 TP, J3 TP, J4 TP, J5 SMA, J6 HF, J7 TP, J8 TP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

Commit message: ADD: pictures and refactored schematic
Routing:
- net GNDS: track 8.40 -> 11.2 mm, vias 45 -> 46
- net GND: track 63.6 -> 60.8 mm, vias 99 -> 98
Other:
- net class Default removed
- board text added: "GaN Class-D Wireless Power Amplifier Lucy Fauth 01/2021 V1.1"
- board text removed: "GaN Class-D Wireless Power Amplifier Niklas Fauth 01/2021 V1.1"
